File: SimpleJoyRx_hw/SimpleJoyRx.sch (KiCad schematic (older format))
At the start: 122 parts

Commit message: + TX sch RC
Parts:
- removed D?: L-C191LBCT, LEDs:LED_0603, symbol LED
- removed R?: 1k, Resistors:RES_0603, symbol R
- removed U?: BT_HC05, Modules:BT_HC0x, symbol BT_HC05
Connections:
- net labels removed: BT_PIO11, BT_RESET, MCURX_BTTX, MCUTX_BTRX
- wire segments 389 -> 369
- no-connect marks 12 -> 11
Other:
- note removed: "Bluetooth"
Changed lines of the file:
@@
 Wire Wire Line
 	13550 14300 13850 14300
-$Comp
-L GND #PWR?
-U 1 1 59D7666F
-P 10200 7700
-F 0 "#PWR?" H 10290 7680 30  0001 C CNN
-F 1 "GND" H 10200 7620 30  0001 C CNN
-F 2 "" H 10200 7700 60  0000 C CNN
-F 3 "" H 10200 7700 60  0000 C CNN
-	1    10200 7700
-	1    0    0    -1
-$EndComp
-$Comp
-L +3.3V #PWR?
-U 1 1 59D76675
-P 10200 7250
-F 0 "#PWR?" H 10200 7210 30  0001 C CNN
-F 1 "+3.3V" H 10280 7280 30  0000 C CNN
-F 2 "" H 10200 7250 60  0000 C CNN
-F 3 "" H 10200 7250 60  0000 C CNN
-	1    10200 7250
-	1    0    0    -1
-$EndComp
-$Comp
-L GND #PWR?
-U 1 1 59D7667B
-P 10700 7700
-F 0 "#PWR?" H 10790 7680 30  0001 C CNN
-F 1 "GND" H 10700 7620 30  0001 C CNN
-F 2 "" H 10700 7700 60  0000 C CNN
-F 3 "" H 10700 7700 60  0000 C CNN
-	1    10700 7700
-	-1   0    0    1
-$EndComp
-$Comp
-L R R?
-U 1 1 59D76683
-P 10450 6950
-F 0 "R?" V 10530 6800 50  0000 C CNN
-F 1 "1k" V 10450 6950 50  0000 C CNN
-F 2 "Resistors:RES_0603" V 10530 7050 28  0001 C CNN
-F 3 "" V 10530 6800 60  0000 C CNN
-F 4 "0.5" V 10630 6900 60  0001 C CNN "Price"
-F 5 "2" V 10730 7000 60  0001 C CNN "SolderPoints"
-	1    10450 6950
-	0    1    -1   0
-$EndComp
-Text Label 8550 7450 0    60   ~ 0
-BT_RESET
-Text Notes 9250 5550 0    60   ~ 0
-Bluetooth
-$Comp
-L LED D?
-U 1 1 59D766A7
-P 10700 7400
-F 0 "D?" H 11000 7550 50  0000 C CNN
-F 1 "L-C191LBCT" H 10620 7540 50  0000 C CNN
-F 2 "LEDs:LED_0603" H 10700 7440 60  0001 C CNN
-F 3 "" H 10800 7540 60  0001 C CNN
-F 4 "2.4" H 10900 7640 60  0001 C CNN "Price"
-F 5 "2" H 11000 7740 60  0001 C CNN "SolderPoints"
-F 6 "http://onelec.ru/products/l-c191lbct" H 10700 7400 60  0001 C CNN "URL"
-F 7 "L-C191LBCT" H 10700 7400 60  0001 C CNN "PN"
-F 8 "Blue" H 10700 7250 39  0000 C CNN "Color"
-	1    10700 7400
-	0    1    1    0
-$EndComp
-$Comp
-L BT_HC05 U?
-U 1 1 59D766BA
-P 9650 7350
-F 0 "U?" H 10000 8250 60  0000 C CNN
-F 1 "BT_HC05" H 9600 8250 60  0000 C CNN
-F 2 "Modules:BT_HC0x" H 9900 8150 60  0001 C CNN
-F 3 "" H 10000 8250 60  0000 C CNN
-F 4 "34" H 10100 8350 60  0001 C CNN "SolderPoints"
-F 5 "" H 10200 8450 60  0001 C CNN "Price"
-	1    9650 7350
-	1    0    0    -1
-$EndComp
-Wire Wire Line
-	10200 7250 10100 7250
-Wire Wire Line
-	10200 7350 10200 7700
-Wire Wire Line
-	10200 7350 10100 7350
-Wire Wire Line
-	10100 7450 10200 7450
-Connection ~ 10200 7450
-Wire Wire Line
-	10700 7700 10700 7600
-Wire Wire Line
-	10700 6950 10700 7200
-Wire Wire Line
-	10200 6950 10100 6950
-Wire Wire Line
-	8550 7450 9200 7450
-Wire Wire Line
-	9200 6900 9200 6950
-Wire Wire Line
-	9200 7100 9200 7050
-Wire Wire Line
-	8550 7250 9200 7250
-Wire Wire Line
-	10100 7550 10200 7550
-Connection ~ 10200 7550
-Wire Wire Line
-	10100 7050 10150 7050
-Wire Wire Line
-	10150 7050 10150 6950
-Connection ~ 10150 6950
-NoConn ~ 9200 7550
-Text Label 8550 7250 0    60   ~ 0
-BT_PIO11
-Text Label 9650 3700 2    60   ~ 0
-MCURX_BTTX
-Text Label 9650 3600 2    60   ~ 0
-MCUTX_BTRX
-Text Label 9650 2400 2    60   ~ 0
-BT_RESET
-Wire Wire Line
-	9650 2400 9000 2400
-Wire Wire Line
-	9650 3700 9000 3700
-Wire Wire Line
-	9650 3600 9000 3600
-Wire Wire Line
-	9650 3800 9000 3800
-Text Label 9650 3800 2    60   ~ 0
-BT_PIO11
-Text Label 8550 6900 0    60   ~ 0
-MCURX_BTTX
-Text Label 8550 7100 0    60   ~ 0
-MCUTX_BTRX
-Wire Wire Line
-	8550 6900 9200 6900
-Wire Wire Line
-	8550 7100 9200 7100
 Wire Notes Line
 	7800 5200 7800 8850
@@
 L DIPx8 SW?
 U 1 1 59D7CD18
-P 6200 6750
-F 0 "SW?" H 6200 7187 60  0000 C CNN
-F 1 "DIPx8" H 6200 7081 60  0000 C CNN
-F 2 "" H 6200 6750 60  0000 C CNN
-F 3 "" H 6200 6750 60  0000 C CNN
-	1    6200 6750
+P 9700 7150
+F 0 "SW?" H 9700 7587 60  0000 C CNN
+F 1 "DIPx8" H 9700 7481 60  0000 C CNN
+F 2 "" H 9700 7150 60  0000 C CNN
+F 3 "" H 9700 7150 60  0000 C CNN
+	1    9700 7150
 	1    0    0    -1
 $EndComp
@@
 L GND #PWR?
 U 1 1 59D82AEF
-P 6600 7400
-F 0 "#PWR?" H 6690 7380 30  0001 C CNN
-F 1 "GND" H 6600 7320 30  0001 C CNN
-F 2 "" H 6600 7400 60  0000 C CNN
-F 3 "" H 6600 7400 60  0000 C CNN
-	1    6600 7400
+P 10100 7800
+F 0 "#PWR?" H 10190 7780 30  0001 C CNN
+F 1 "GND" H 10100 7720 30  0001 C CNN
+F 2 "" H 10100 7800 60  0000 C CNN
+F 3 "" H 10100 7800 60  0000 C CNN
+	1    10100 7800
 	1    0    0    -1
 $EndComp
 Wire Wire Line
-	6600 6600 6600 7400
+	10100 7000 10100 7800
 Wire Wire Line
-	6600 7300 6500 7300
+	10100 7700 10000 7700
 Wire Wire Line
-	6500 7200 6600 7200
-Connection ~ 6600 7300
+	10000 7600 10100 7600
+Connection ~ 10100 7700
 Wire Wire Line
-	6500 7100 6600 7100
-Connection ~ 6600 7200
+	10000 7500 10100 7500
+Connection ~ 10100 7600
 Wire Wire Line
-	6500 7000 6600 7000
-Connection ~ 6600 7100
+	10000 7400 10100 7400
+Connection ~ 10100 7500
 Wire Wire Line
-	6500 6900 6600 6900
-Connection ~ 6600 7000
+	10000 7300 10100 7300
+Connection ~ 10100 7400
 Wire Wire Line
-	6500 6800 6600 6800
-Connection ~ 6600 6900
+	10000 7200 10100 7200
+Connection ~ 10100 7300
 Wire Wire Line
-	6500 6700 6600 6700
-Connection ~ 6600 6800
+	10000 7100 10100 7100
+Connection ~ 10100 7200
 Wire Wire Line
-	6500 6600 6600 6600
-Connection ~ 6600 6700
-Text Label 5650 6600 0    60   ~ 0
+	10000 7000 10100 7000
+Connection ~ 10100 7100
+Text Label 9150 7000 0    60   ~ 0
 DIP1
-Text Label 5650 6700 0    60   ~ 0
+Text Label 9150 7100 0    60   ~ 0
 DIP2
-Text Label 5650 6800 0    60   ~ 0
+Text Label 9150 7200 0    60   ~ 0
 DIP3
-Text Label 5650 6900 0    60   ~ 0
+Text Label 9150 7300 0    60   ~ 0
 DIP4
-Text Label 5650 7000 0    60   ~ 0
+Text Label 9150 7400 0    60   ~ 0
 DIP5
-Text Label 5650 7100 0    60   ~ 0
+Text Label 9150 7500 0    60   ~ 0
 DIP6
-Text Label 5650 7200 0    60   ~ 0
+Text Label 9150 7600 0    60   ~ 0
 DIP7
-Text Label 5650 7300 0    60   ~ 0
+Text Label 9150 7700 0    60   ~ 0
 DIP8
 Wire Wire Line
-	5650 6600 5900 6600
+	9150 7000 9400 7000
 Wire Wire Line
-	5900 6700 5650 6700
+	9400 7100 9150 7100
 Wire Wire Line
-	5650 6800 5900 6800
+	9150 7200 9400 7200
 Wire Wire Line
-	5900 6900 5650 6900
+	9400 7300 9150 7300
 Wire Wire Line
-	5650 7000 5900 7000
+	9150 7400 9400 7400
 Wire Wire Line
-	5900 7100 5650 7100
+	9400 7500 9150 7500
 Wire Wire Line
-	5650 7200 5900 7200
+	9150 7600 9400 7600
 Wire Wire Line
-	5900 7300 5650 7300
+	9400 7700 9150 7700
 Text Label 5500 1700 0    60   ~ 0
 DIP1
@@
 Wire Wire Line
 	5750 2400 5500 2400
-Text Notes 5950 5550 0    60   ~ 0
+Text Notes 9450 5950 0    60   ~ 0
 DIP Switch
 $Comp

Commit message: + RX sch
Parts:
- removed C? (x2): 18pF, Capacitors:CAP_0603, symbol C
- removed L?: BLM15AG102, Inductors:IND_0402, symbol L
- removed Q?: IRF9310, SO_DIL_TSSOP:SO8_150MIL, symbol P_8PIN
- removed R?: 1k, Resistors:RES_0603, symbol R
- removed XTAL?: 12MHz, Quartz:0503x4-4, symbol CRYSTAL_H
- added D1: L-C191KGCT, LEDs:LED_0603, symbol LED
- added D2: L-C191LBCT, LEDs:LED_0603, symbol LED
- added unit 1 of Q1
- added R3, R4, R5: 1k, Resistors:RES_0603, symbol R
- gave numbers to parts that had none: 113
Connections:
- net labels removed: PWR_UNST_ALWAYS, PwrMCU
- wire segments 369 -> 362
- no-connect marks 11 -> 26
Other:
- note added: "Link"
- note added: "Power\nconnector"
- note added: "USB Detect"
- note removed: "Battery\nconnector"

Commit message: * DRV8835 for 4 channels
Parts:
- removed C13, C14, C24, C35: 100u 6V3, Capacitors:CAP_1206, symbol C
- removed C15, C16, C26, C39: 0.1u, Capacitors:CAP_0603, symbol C
- removed D5, D6, D7, D9: PMEG2020, Diodes:SOD323, symbol D_Shottky
- removed Q2, Q3, Q5, Q7: IRLML0030, SOT:SOT23-3, symbol N_3PIN
- removed R13, R15, R7, R8: 56k, Resistors:RES_0603, symbol R
- removed XL10, XL15, XL6, XL8: PLS2, Connectors:PLS-2, symbol CONN_2
- added C? (x4): 0.1u, Capacitors:CAP_0603, symbol C
- added C? (x4): 100u 6V3, Capacitors:CAP_1206, symbol C
- added DA? (x2): DRV8835, QFN_DFN:WSON12, symbol DRV8835
- added XL? (x4): PLS2, Connectors:PLS-2, symbol CONN_2
Connections:
- net labels added: DIR1, DIR2, DIR3, DIR4, MOTORA1, MOTORA2, MOTORB1, MOTORB2, MOTORC1, MOTORC2, MOTORD1, MOTORD2
- net labels removed: PWM_OUT1, PWM_OUT2, PWM_OUT3, PWM_OUT4
- wire segments 362 -> 354
- no-connect marks 26 -> 22
Other:
- note added: "Motor drivers\nLogic high sets PH/EN mode"

Commit message: RX PCB 2x5
Parts:
- removed C10: 1000u, Capacitors:CAP_10Rx16_HOR, symbol CP
- removed HOLE3, HOLE4: HOLE_METALLED, PCB:Hole3_5_out6mm, symbol HOLE_METALLED
- removed XL13: CONN_1, Connectors:PLS-1Rnd, symbol CONN_1
- added C12, C13: 100u 6V3, Capacitors:CAP_1206, symbol C
- added RP1, RP2, RP3, RP4: REFPOINT, PCB:REF_POINT_1MM, symbol REFPOINT
- added XL18: CONN_1, Connectors:PLS-1Rnd, symbol CONN_1
- HOLE1, HOLE2: footprint PCB:Hole3_5_out6mm -> PCB:Hole2d4_out4d5mm
- SW1: renamed from SW2; footprint (none) -> BtnsSwitches:DIP_SMD_X8; Price (none) -> 27; SolderPoints (none) -> 16; URL (none) -> http://www.zip-2002.ru/kommutatsiya/dip_pereklyuchateli/712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
- SW3: value SS-12F23 -> 1P2T; footprint BtnsSwitches:SW_SS-12F23 -> BtnsSwitches:SW_SS-1P2T; PN Q-563(SS-12F23) -> (none); Price 15 -> 10; URL http://www.quartz1.com/price/model.php?group=1505&ext=563 -> (none)
- XL10: renamed from XL5; footprint (none) -> Connectors:PLS-3
- XL11: renamed from XL9; footprint (none) -> Connectors:PLS-3
- XL12: renamed from XL14; footprint (none) -> Connectors:PLS-3
- XL13: renamed from XL11; footprint (none) -> Connectors:PLS-3
- XL16: footprint (none) -> Connectors:PLS-3
- XL9: renamed from XL7; footprint (none) -> Connectors:PLS-3
- gave numbers to parts that had none: 14
- renumbered C12 to C20, C11 to C21, C30 to C23, C17 to C24, C18 to C25, C19 to C26, C20 to C27, C21 to C28, C23 to C29, C25 to C30, C27 to C31, C28 to C32, C29 to C33, C31 to C34, C32 to C35, C33 to C36, C34 to C37, C36 to C38, C37 to C39, C38 to C40, C40 to C41, C41 to C42, C42 to C43, D8 to D5, D10 to D6, DA2 to DA3, DA1 to DA4, DA4 to DA5, DA3 to DA7, DA5 to DA8, DA7 to DA9, Q4 to Q2, Q6 to Q3, Q8 to Q4, R12 to R10, R14 to R11, R16 to R12, R5 to R3, R3 to R4, R4 to R5, R9 to R7, R10 to R8, R11 to R9, SW1 to SW2, XL12 to XL14, XL4 to XL8
Connections:
- wire segments 354 -> 360
- no-connect marks 22 -> 18

Commit message: RX layout done
Parts:
- HOLE1, HOLE2: footprint PCB:Hole2d4_out4d5mm -> PCB:Hole3d3_out5d5mm
- XL2: value USB_MINI_B -> USB_MICRO; footprint Connectors:USBmicro_MOLEX_WM17142 -> Connectors:USBmicro_MOLEX_1050170001
Connections:
- wire segments 360 -> 359
Changed lines of the file:
@@
 P 1200 2900
 F 0 "XL2" H 1000 3350 60  0000 C CNN
-F 1 "USB_MINI_B" H 1100 3250 60  0000 C CNN
-F 2 "Connectors:USBmicro_MOLEX_WM17142" H 1200 2900 60  0001 C CNN
+F 1 "USB_MICRO" H 1100 3250 60  0000 C CNN
+F 2 "Connectors:USBmicro_MOLEX_1050170001" H 1200 2900 60  0001 C CNN
 F 3 "" H 1200 2900 60  0000 C CNN
 	1    1200 2900
@@
 L GND #PWR0104
 U 1 1 59D4DD4F
-P 20800 14700
-F 0 "#PWR0104" H 20890 14680 30  0001 C CNN
-F 1 "GND" H 20800 14620 30  0001 C CNN
-F 2 "" H 20800 14700 60  0001 C CNN
-F 3 "" H 20800 14700 60  0001 C CNN
-	1    20800 14700
-	1    0    0    -1
+P 20800 14300
+F 0 "#PWR0104" H 20890 14280 30  0001 C CNN
+F 1 "GND" H 20800 14220 30  0001 C CNN
+F 2 "" H 20800 14300 60  0001 C CNN
+F 3 "" H 20800 14300 60  0001 C CNN
+	1    20800 14300
+	0    1    1    0
 $EndComp
 $Comp
@@
 F 0 "HOLE1" H 20050 14300 60  0000 C CNN
 F 1 "HOLE_METALLED" H 19850 14350 60  0001 C CNN
-F 2 "PCB:Hole2d4_out4d5mm" H 19800 14150 60  0001 C CNN
+F 2 "PCB:Hole3d3_out5d5mm" H 19800 14150 60  0001 C CNN
 F 3 "" H 19900 14250 60  0001 C CNN
 F 4 "0" H 20000 14350 60  0001 C CNN "Price"
@@
 F 0 "HOLE2" H 20050 14550 60  0000 C CNN
 F 1 "HOLE_METALLED" H 19850 14600 60  0001 C CNN
-F 2 "PCB:Hole2d4_out4d5mm" H 19800 14400 60  0001 C CNN
+F 2 "PCB:Hole3d3_out5d5mm" H 19800 14400 60  0001 C CNN
 F 3 "" H 19900 14500 60  0001 C CNN
 F 4 "0" H 20000 14600 60  0001 C CNN "Price"
@@
 	9000 900  9100 900
 Wire Wire Line
-	20800 14300 20800 14700
-Wire Wire Line
 	17450 14100 17550 14100
 Connection ~ 17100 14950
@@
 Wire Wire Line
 	20800 14300 20700 14300
+$Comp
+L GNDPWR #PWR?
+U 1 1 59DB0108
+P 20800 14550
+F 0 "#PWR?" H 20800 14600 40  0001 C CNN
+F 1 "GNDPWR" H 20800 14470 40  0001 C CNN
+F 2 "" H 20800 14550 60  0000 C CNN
+F 3 "" H 20800 14550 60  0000 C CNN
+	1    20800 14550
+	0    -1   -1   0
+$EndComp
 Wire Wire Line
 	20700 14550 20800 14550
-Connection ~ 20800 14550
 $EndSCHEMATC

Commit message: + Antenna
Parts:
- ANT1: footprint Radio:ANT_868_SEIDHE -> Radio:ANT_868_24x30
Changed lines of the file:
@@
 F 0 "ANT1" H 20000 1950 60  0000 C CNN
 F 1 "ANT_PCB_MONO" H 20250 1850 60  0000 C CNN
-F 2 "Radio:ANT_868_SEIDHE" H 19900 1850 60  0001 C CNN
+F 2 "Radio:ANT_868_24x30" H 19900 1850 60  0001 C CNN
 F 3 "" H 20000 1950 60  0001 C CNN
 F 4 "0" H 20100 2050 60  0001 C CNN "Price"

Commit message: RX PCB seems done
Parts:
- added Logo2: Logo, Pictures:Livetronic27x9, symbol Logo
- Logo1: footprint Pictures:Ostranna_12d7_10d1 -> Pictures:Ostranna_8x8
Changed lines of the file:
@@
 L Logo Logo1
 U 1 1 59D4DD55
-P 19150 14300
-F 0 "Logo1" H 19428 14353 60  0000 L CNN
-F 1 "Logo" H 19428 14247 60  0000 L CNN
-F 2 "Pictures:Ostranna_12d7_10d1" H 19150 14300 60  0001 C CNN
-F 3 "" H 19150 14300 60  0000 C CNN
-	1    19150 14300
+P 19150 13450
+F 0 "Logo1" H 19428 13503 60  0000 L CNN
+F 1 "Logo" H 19428 13397 60  0000 L CNN
+F 2 "Pictures:Ostranna_8x8" H 19150 13450 60  0001 C CNN
+F 3 "" H 19150 13450 60  0000 C CNN
+	1    19150 13450
 	1    0    0    -1
 $EndComp
@@
 F 5 "0.5" H 21850 9100 60  0001 C CNN "Price"
 	1    21850 9100
-	1    0    0    1
+	1    0    0    -1
 $EndComp
 $Comp
@@
 F 5 "0.5" H 18900 9050 60  0001 C CNN "Price"
 	1    18900 9050
-	1    0    0    1
+	1    0    0    -1
 $EndComp
 $Comp
@@
 	20800 14300 20700 14300
 $Comp
-L GNDPWR #PWR?
+L GNDPWR #PWR0127
 U 1 1 59DB0108
 P 20800 14550
-F 0 "#PWR?" H 20800 14600 40  0001 C CNN
+F 0 "#PWR0127" H 20800 14600 40  0001 C CNN
 F 1 "GNDPWR" H 20800 14470 40  0001 C CNN
 F 2 "" H 20800 14550 60  0000 C CNN
@@
 Wire Wire Line
 	20700 14550 20800 14550
+$Comp
+L Logo Logo2
+U 1 1 59DBA4A2
+P 19150 14350
+F 0 "Logo2" H 19428 14403 60  0000 L CNN
+F 1 "Logo" H 19428 14297 60  0000 L CNN
+F 2 "Pictures:Livetronic27x9" H 19150 14350 60  0001 C CNN
+F 3 "" H 19150 14350 60  0000 C CNN
+	1    19150 14350
+	1    0    0    -1
+$EndComp
 $EndSCHEMATC

Commit message: TX layout started
Parts:
- added Logo3: Logo, Pictures:Livetronic13x4, symbol Logo
