File: SimpleJoyRx_hw/SimpleJoyRx.sch (KiCad schematic (older format))
At the start: 113 parts, among them Q1 IRF9358, Q2 2N7002, Q3 IRLML0030, Q4 IRLML0030, SW1 DIPx8, SW2 BUTTON, SW3 1P2T, U1 USBLC6

Commit message: + Antennas matched
Parts:
- C35: value * -> 2.4pF
- C40: value * -> DoNotMount
- L2: value * -> 1.2nH
Changed lines of the file:
@@
 LIBS:standard_logic
 LIBS:modules
+LIBS:Sensors
 LIBS:SimpleJoyRx-cache
 EELAYER 26 0
@@
 P 18750 1700
 F 0 "L2" V 18650 1560 40  0000 C CNN
-F 1 "*" V 18650 1700 40  0000 C CNN
+F 1 "1.2nH" V 18650 1700 40  0000 C CNN
 F 2 "Inductors:IND_0402" V 18810 1710 40  0001 C CNN
 F 3 "" V 18650 1560 60  0001 C CNN
@@
 P 18400 2200
 F 0 "C35" H 18300 2100 50  0000 L CNN
-F 1 "*" H 18300 2300 50  0000 L CNN
+F 1 "2.4pF" H 18300 2300 50  0000 L CNN
 F 2 "Capacitors:CAP_0402" V 18500 2050 28  0001 C BNN
 F 3 "" H 18300 2100 60  0001 C CNN
@@
 P 19100 2200
 F 0 "C40" H 19000 2100 50  0000 L CNN
-F 1 "*" H 19000 2300 50  0000 L CNN
+F 1 "DoNotMount" H 18900 2300 50  0000 L CNN
 F 2 "Capacitors:CAP_0402" V 19200 2050 28  0001 C BNN
 F 3 "" H 19000 2100 60  0001 C CNN

Commit message: + RX v2
Parts:
- removed C22, C23, C29, C34: 0.1u, Capacitors:CAP_0603, symbol C
- removed DA3, DA4, DA5, DA6, DA8, DA9: MC74VHC1, SOT:SOT23-5, symbol MC74VHC1
- added DA3: MCP1700, SOT:SOT23-3A, symbol MCP1700
- added XL15, XL19, XL20, XL21: PLS3, Connectors:PLS-3, symbol CONN_3
- BLN1: Price (none) -> 45
- C1, C20, C21, C32, R10, R2, R7, R9: Price (none) -> 0.5; SolderPoints (none) -> 2
- DA7: footprint SOT:SOT23-3 -> SOT:SOT23-3A
- L1: Price (none) -> 1; SolderPoints (none) -> 2
- Logo1, Logo2, Logo3, RP1, RP2, RP3, RP4, XL18: Price (none) -> 0; SolderPoints (none) -> 0
- Q2: Price (none) -> 1.6
- SW2: value BUTTON -> IT-1187A; PN (none) -> IT-1187A; Price (none) -> 4; SolderPoints (none) -> 4
- SW3: SolderPoints (none) -> 3
- U1: SolderPoints (none) -> 6
- XL1: Price (none) -> 1; SolderPoints (none) -> 6; SolderPointsDIP 6 -> (none)
- XL14, XL17, XL4, XL5, XL6, XL7: SolderPoints (none) -> 2
- XL2: PN (none) -> 47491-0001; Price (none) -> 46; SolderPoints (none) -> 9
- XL3: Price (none) -> 2; SolderPoints (none) -> 2
- XL8: value CONN_2 -> PLS2; Price (none) -> 0.5; SolderPoints (none) -> 2; SolderPointsDip (none) -> 2
Connections:
- net labels added: A1, A2, A3, A4, VAA
- wire segments 359 -> 346
- no-connect marks 18 -> 14
Other:
- note added: "Analog inputs"
