File: SimpleJoyRx_hw/SimpleJoyRx.sch (KiCad schematic (older format))
At the start: 107 parts, among them Q1 IRF9358, Q2 2N7002, Q3 IRLML0030, Q4 IRLML0030, SW1 DIPx8, SW2 IT-1187A, SW3 SS-12F23

Commit message: * rPkt format changed * Rx v3 done Seems working
Parts:
- removed C38: 100u 6V3, Capacitors:CAP_1206, symbol SimpleJoyRx-rescue:C-RESCUE-SimpleJoyRx
- removed C41: 0.1u, Capacitors:CAP_0603, symbol SimpleJoyRx-rescue:C-RESCUE-SimpleJoyRx
- removed D5, D6: PMEG2020, Diodes:SOD323, symbol SimpleJoyRx-rescue:D_Shottky-RESCUE-SimpleJoyRx
- removed Q2: 2N7002, SOT:SOT23-3, symbol SimpleJoyRx-rescue:N_3PIN-RESCUE-SimpleJoyRx
- removed Q3, Q4: IRLML0030, SOT:SOT23-3, symbol SimpleJoyRx-rescue:N_3PIN-RESCUE-SimpleJoyRx
- removed R7: 100k, Resistors:RES_0603, symbol SimpleJoyRx-rescue:R-RESCUE-SimpleJoyRx
- removed XL14: PLS2, Connectors:PLS-2, symbol SimpleJoyRx-rescue:CONN_2-RESCUE-SimpleJoyRx
- added C22, C34: 0.1u, Capacitors:CAP_0603, symbol SimpleJoyRx-rescue:C-RESCUE-SimpleJoyRx
- added C23, C29: 100u 6V3, Capacitors:CAP_1206, symbol SimpleJoyRx-rescue:C-RESCUE-SimpleJoyRx
- added DA4: DRV8835, QFN_DFN:WSON12, symbol SimpleJoyRx-rescue:DRV8835-RESCUE-SimpleJoyRx
- added XL14: CONN_4, Connectors:PLS-4, symbol Connectors_kl:CONN_4
- added XL22: PLS2, Connectors:PLS-2, symbol SimpleJoyRx-rescue:CONN_2-RESCUE-SimpleJoyRx
- C30: value 100u 6V3 -> 0.1u; footprint Capacitors:CAP_1206 -> Capacitors:CAP_0603; PN CL31A107MQHNNNE -> (none); Price 7 -> 0.5
- C31: value 0.1u -> 10u; Price 0.5 -> 4
- R11, R12: value 56k -> 10k
- SW3: URL (none) -> http://www.quartz1.com/price/model.php?akt=3843.17
Connections:
- net labels added: DIR5, DIR6, MOTORE1, MOTORE2, MOTORF1, MOTORF2, SCL, SDA
- net labels removed: MEASURE_EN, PWM_OUT5, PWM_OUT6
- wire segments 423 -> 431
- no-connect marks 14 -> 11
Other:
- note added: "I2C connector"
- moved on the sheet: R10, R9
