File: SimpleJoyRx_hw/SimpleJoyRx.kicad_sch (KiCad schematic)
At the start: 105 parts, among them Q1 IRF9358, SW1 DIPx8, SW2 IT-1187A, SW3 SS-12F23

Commit message: + RX L476fw os
Parts:
- added DD?: STM32L476Rx, LQFP_TQFP:LQFP64, symbol st_kl:STM32L476Rx
Changed lines of the file:
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@@
     (pin "2")
+  )
+  (symbol (lib_id "st_kl:STM32L476Rx") (at 189.23 -53.34 0) (unit 1)
+    (in_bom yes) (on_board yes)
+    (property "Reference" "DD?" (id 0) (at 177.8 -92.71 0)
+      (effects (font (size 1.524 1.524)))
+    )
+    (property "Value" "STM32L476Rx" (id 1) (at 194.31 -92.71 0)
+      (effects (font (size 1.524 1.524)))
+    )
+    (property "Footprint" "LQFP_TQFP:LQFP64" (id 2) (at 186.69 -98.425 0)
+      (effects (font (size 1.524 1.524)) hide)
+    )
+    (property "Datasheet" "" (id 3) (at 189.23 -53.34 0)
+      (effects (font (size 1.524 1.524)))
+    )
+    (property "SolderPoints" "64" (id 4) (at 180.34 -95.25 0)
+      (effects (font (size 1.524 1.524)) hide)
+    )
+    (property "Price" "290" (id 5) (at 182.88 -97.79 0)
+      (effects (font (size 1.524 1.524)) hide)
+    )
+    (property "PN" "STM32L476RCT6" (id 6) (at 185.42 -100.33 0)
+      (effects (font (size 1.524 1.524)) hide)
+    )
+    (pin "1")
+    (pin "10")
+    (pin "11")
+    (pin "12")
+    (pin "13")
+    (pin "14")
+    (pin "15")
+    (pin "16")
+    (pin "17")
+    (pin "18")
+    (pin "19")
+    (pin "2")
+    (pin "20")
+    (pin "21")
+    (pin "22")
+    (pin "23")
+    (pin "24")
+    (pin "25")
+    (pin "26")
+    (pin "27")
+    (pin "28")
+    (pin "29")
+    (pin "3")
+    (pin "30")
+    (pin "31")
+    (pin "32")
+    (pin "33")
+    (pin "34")
+    (pin "35")
+    (pin "36")
+    (pin "37")
+    (pin "38")
+    (pin "39")
+    (pin "4")
+    (pin "40")
+    (pin "41")
+    (pin "42")
+    (pin "43")
+    (pin "44")
+    (pin "45")
+    (pin "46")
+    (pin "47")
+    (pin "48")
+    (pin "49")
+    (pin "5")
+    (pin "50")
+    (pin "51")
+    (pin "52")
+    (pin "53")
+    (pin "54")
+    (pin "55")
+    (pin "56")
+    (pin "57")
+    (pin "58")
+    (pin "59")
+    (pin "6")
+    (pin "60")
+    (pin "61")
+    (pin "62")
+    (pin "63")
+    (pin "64")
+    (pin "7")
+    (pin "8")
+    (pin "9")
   )
   (sheet_instances
@@
       (reference "DD2") (unit 1) (value "CC1101") (footprint "QFN_DFN:QFN20")
     )
+    (path "/b975ded2-97d3-450f-999c-18c2890e9341"
+      (reference "DD?") (unit 1) (value "STM32L476Rx") (footprint "LQFP_TQFP:LQFP64")
+    )
     (path "/00000000-0000-0000-0000-000059d7fc35"
