File: SimpleJoyTx_hw/SimpleJoyTx.kicad_pcb (KiCad board)
At the start: 2 copper layers, 108 x 63 mm, 79 parts, among them J1 Joystick, J2 Joystick, Q1 2N7002, SW1 IT-1187A, SW2 DIPx8, SW3 SWITCH, SW4 IT-1187A, SW5 IT-1187A, SW6 IT-1187A, SW7 IT-1187A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

Commit message: + Layout + antenna
Parts:
- added D4: L-C191KGCT, LEDs:LED_0603, F.Cu at (126.0, 80.0)
- added D5: L-C191LBCT, LEDs:LED_0603, F.Cu at (126.0, 75.0)
- added Logo3: Logo, Pictures:Livetronic27x9, B.Cu at (181.0, 53.0)
- added R12: 1k, Resistors:RES_0603, F.Cu at (130.0, 80.0)
- added R13: 1k, Resistors:RES_0603, F.Cu at (130.0, 75.0)
- ANT1: value ANT_PCB_MONO -> ANT_PCB_MONO_2PIN; footprint Radio:ANT_868_SEIDHE -> Radio:ANT_868_IFA_SIMPLEJOY
- SW1: moved to B.Cu
- SW3: footprint BtnsSwitches:SW_SS-1P2T -> BtnsSwitches:SW_SS-12F23; moved to B.Cu
- moved Logo1 214.2 mm to (117.0, 78.0)
- moved L4 205.5 mm to (135.1, 60.3), turned to 270 degrees
- moved C20 205.0 mm to (134.6, 62.0), turned to 180 degrees
- moved C23 203.9 mm to (135.7, 58.6)
- moved C17 203.6 mm to (129.9, 71.4), turned to 180 degrees
- moved C25 201.1 mm to (129.9, 69.8), turned to 180 degrees
- moved C24 198.6 mm to (135.8, 74.2), turned to 270 degrees
- moved C14 198.1 mm to (143.2, 65.2)
- moved C19 197.5 mm to (132.3, 63.9), turned to 180 degrees
- moved XTAL2 197.3 mm to (143.2, 68.3), turned to 90 degrees
- moved D3 197.2 mm to (135.6, 112.6)
- moved R9 196.2 mm to (129.9, 68.2), turned to 180 degrees
- moved C13 196.1 mm to (139.0, 100.8)
- moved DA1 193.6 mm to (139.0, 104.0)
- moved C12 192.1 mm to (135.2, 105.0), turned to 180 degrees
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Connections:
- DD1 pad 2: (no net) -> Net-(DD1-Pad2)
- DD1 pad 3: (no net) -> Net-(DD1-Pad3)
- DD1 pad 4: (no net) -> Net-(DD1-Pad4)
- DD1 pad 54: (no net) -> Net-(DD1-Pad54)
- DD1 pad 7: (no net) -> Net-(DD1-Pad7)
- DD2 pad 3: (no net) -> Net-(DD2-Pad3)
- HOLE1 pad H: (no net) -> GND
- HOLE2 pad H: (no net) -> GND
- HOLE3 pad H: (no net) -> GND
- HOLE4 pad H: (no net) -> GND
- HOLE5 pad H: Net-(HOLE5-PadH) -> GND
- HOLE6 pad H: Net-(HOLE6-PadH) -> GND
- HOLE7 pad H: Net-(HOLE7-PadH) -> GND
- HOLE8 pad H: Net-(HOLE8-PadH) -> GND
- J1 pad 11: (no net) -> Net-(J1-Pad11)
- J1 pad 12: (no net) -> Net-(J1-Pad12)
- J1 pad 3: (no net) -> Net-(J1-Pad3)
- J1 pad 7: (no net) -> Net-(J1-Pad7)
- J2 pad 11: (no net) -> Net-(J2-Pad11)
- J2 pad 12: (no net) -> Net-(J2-Pad12)
- J2 pad 3: (no net) -> Net-(J2-Pad3)
- J2 pad 7: (no net) -> Net-(J2-Pad7)
- SW3 pad 3: (no net) -> Net-(SW3-Pad3)
- XL2 pad 1: (no net) -> +3.3V
- XL3 pad H2: (no net) -> Net-(XL3-PadH2)
- XL3 pad H3: (no net) -> Net-(XL3-PadH3)
Other:
- board size 108 x 63 mm -> 108 x 66 mm
- net class Default: trace_width 0.25 -> 0.2; via_dia 0.8 -> 0.9
- net class Wide added: clearance 0.2, trace_width 0.5, via_dia 0.9, via_drill 0.4

Commit message: + SimpleJoy TX * Leg 63 bug fixed
Parts:
- added RP1: REFPOINT, PCB:REF_POINT_1MM, F.Cu at (118.0, 113.2)
- added RP2: REFPOINT, PCB:REF_POINT_1MM, B.Cu at (118.0, 113.2)
- added RP3: REFPOINT, PCB:REF_POINT_1MM, B.Cu at (216.4, 50.8)
- added RP4: REFPOINT, PCB:REF_POINT_1MM, F.Cu at (216.4, 50.8)
- moved Logo3 17.8 mm to (163.2, 52.6)
- moved Logo2 17.0 mm to (162.0, 54.0)
- moved C15 6.30 mm to (143.2, 65.2)
- moved C14 6.20 mm to (143.2, 71.4), turned to 180 degrees
- moved C9 2.49 mm to (168.7, 72.9)
- moved C7 0.50 mm to (167.9, 90.2)
- moved C2 0.40 mm to (153.4, 85.2)
- moved C22 0.20 mm to (140.2, 68.4)
- moved BLN1 0.10 mm to (135.9, 63.7)
- moved C20 0.10 mm to (134.7, 62.0)
- moved L4 0.10 mm to (135.2, 60.3)
Connections:
- DD1 pad 62: GND -> /BTN_J2
- DD1 pad 63: (no net) -> GND
Routing:
- net GND: track 0.00 -> 1348.2 mm, vias 0 -> 238
- net +3.3V: track 0.00 -> 305.9 mm, vias 0 -> 9
- net /PWR_UNST_ALWAYS: track 0.00 -> 63.7 mm, vias 0 -> 1
- net Net-(DD1-Pad60): track 0.00 -> 63.2 mm, vias 0 -> 3
- net VCC: track 0.00 -> 61.7 mm, vias 0 -> 6
- net /ADC2: track 0.00 -> 61.3 mm, vias 0 -> 2
- net /ADC0: track 0.00 -> 59.4 mm, vias 0 -> 1
- net /ADC3: track 0.00 -> 57.9 mm, vias 0 -> 2
- net /ADC4: track 0.00 -> 56.4 mm
- net /5V_USB: track 0.00 -> 56.0 mm, vias 0 -> 2
- net /BTN_J1: track 0.00 -> 48.5 mm, vias 0 -> 2
- net /ADC1: track 0.00 -> 45.6 mm, vias 0 -> 1
- net /BTN_J2: track 0.00 -> 44.7 mm, vias 0 -> 1
- net /MCURX_BTTX: track 0.00 -> 44.4 mm
- net /ADC5: track 0.00 -> 43.8 mm, vias 0 -> 1
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- added copper zone on B.Cu, net GND
- added copper zone on F.Cu, net GND
Other:
- outline, holes or cut-outs redrawn
- rule pad_to_mask_clearance: 0.2 -> 0.1
- board text added: "1.0"
- board text added: "B"
- board text added: "BT"
- board text added: "Bootloader"
- board text added: "Debug"
- board text added: "Display"
- board text added: "G"
- board text added: "GND"
- board text added: "Link"
- board text added: "Power"
- board text added: "SimpleJoy TX"

Commit message: TX: USB and switch moved to edges. Sent to production.
Parts:
- moved Logo1 76.4 mm to (192.1, 63.7)
- moved D1 36.7 mm to (217.0, 86.9), turned to 270 degrees
- moved XL3 36.7 mm to (212.4, 79.0), turned to 180 degrees
- moved SW3 34.4 mm to (116.2, 79.2), turned to 90 degrees
- moved R3 31.9 mm to (214.5, 86.0), turned to 180 degrees
- moved C12 29.1 mm to (121.5, 79.3), turned to 90 degrees
- moved C13 28.6 mm to (124.8, 76.0)
- moved DA1 28.6 mm to (124.8, 79.2)
- moved C1 26.9 mm to (208.8, 86.9), turned to 90 degrees
- moved U1 26.5 mm to (207.0, 81.8), turned to 180 degrees
- moved D4 14.1 mm to (112.2, 83.0)
- moved D5 13.8 mm to (112.2, 75.2)
- moved U2 12.0 mm to (190.0, 79.6)
- moved SW1 9.70 mm to (193.4, 110.6), turned to 180 degrees
- moved R12 9.68 mm to (120.8, 83.0)
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Routing:
- net GND: track 1348.2 -> 1270.7 mm, vias 238 -> 225
- net /PWR_UNST_ALWAYS: track 63.7 -> 135.8 mm
- net +3.3V: track 305.9 -> 269.5 mm, vias 9 -> 11
- net /5V_USB: track 56.0 -> 85.5 mm
- net /D-: track 29.9 -> 53.2 mm
- net /D+: track 30.3 -> 51.1 mm
- net Net-(DD1-Pad60): track 63.2 -> 51.5 mm
- net /BT_PIO11: track 39.7 -> 28.8 mm
- net Net-(DD1-Pad2): track 39.0 -> 48.3 mm
- net Net-(DD1-Pad3): track 38.4 -> 47.1 mm
- net /MCUTX_BTRX: track 42.8 -> 36.7 mm
- net /MCURX_BTTX: track 44.4 -> 38.4 mm
- net Net-(R3-Pad2): track 31.6 -> 37.4 mm
- net Net-(D4-PadA): track 2.49 -> 7.46 mm
- net Net-(D5-PadA): track 2.49 -> 7.21 mm
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Other:
- outline, holes or cut-outs redrawn
- net class Default: trace_width 0.2 -> 0.25

Commit message: Proceeding
Parts:
- added C26: 100pF, Capacitors:CAP_0402, F.Cu at (163.4, 32.2)
- C20: value * -> 2pF
- C23: value * -> DoNotMount
- DA1: footprint SOT:SOT23-3 -> SOT:SOT23-3A
- L3: value BLM15AG102SN1 -> BLM15AG102
- L4: value * -> 1.2nH
- XL1: value PLS-8 -> PBS-8
- moved HOLE3 101.3 mm to (113.3, 111.6), turned to 270 degrees
- moved HOLE2 101.2 mm to (113.3, 10.4), turned to 270 degrees
- moved XL4 98.9 mm to (117.9, 113.6), turned to 270 degrees
- moved RP1 98.4 mm to (111.7, 15.0), turned to 270 degrees
- moved RP2 98.4 mm to (111.7, 15.0), turned to 270 degrees
- moved D1 83.5 mm to (138.0, 114.0), turned to 180 degrees
- moved D3 83.3 mm to (112.3, 32.6), turned to 270 degrees
- moved SW1 81.6 mm to (114.3, 90.4), turned to 90 degrees
- moved D2 81.1 mm to (114.1, 32.6), turned to 270 degrees
- moved L1 80.6 mm to (112.5, 36.4), turned to 270 degrees
- moved R3 79.8 mm to (138.9, 111.5), turned to 90 degrees
- moved D4 79.6 mm to (141.9, 9.20), turned to 90 degrees
- moved R5 78.6 mm to (114.1, 36.4), turned to 270 degrees
- moved J2 78.3 mm to (127.9, 103.0), turned to 270 degrees
- moved J1 78.2 mm to (127.9, 19.0), turned to 90 degrees
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Connections:
- BLN1 pad 1: /ANT1 -> Net-(BLN1-Pad1)
- R10 pad 1: +BATT -> /BAT_MEAS
- R10 pad 2: /BAT_MEAS -> +BATT
- R11 pad 1: /BAT_MEAS -> Net-(Q1-Pad3)
- R11 pad 2: Net-(Q1-Pad3) -> /BAT_MEAS
Routing:
- net /BT_RESET: track 30.2 -> 23.1 mm
- net GND: track 1270.7 -> 1267.0 mm
- net VCC: track 60.3 -> 63.1 mm
- net +3.3V: track 269.5 -> 270.8 mm
- net Net-(BLN1-Pad1): track 0.00 -> 1.31 mm
- net Net-(Q1-Pad3): track 1.83 -> 3.10 mm
- net /PWR_UNST_ALWAYS: track 135.8 -> 136.8 mm
- net /ANT2: track 9.45 -> 10.0 mm
Other:
- board size 108 x 66 mm -> 66 x 108 mm
- board text added: "1.1"
- board text added: "A"
- board text added: "C"
- board text added: "D"
- board text added: "L"
- board text added: "OFF"
- board text added: "ON"
- board text removed: "1.0"
