File: SimpleJoyTx_hw/SimpleJoyTx.sch (KiCad schematic (older format))
At the start: 59 parts

Commit message: + TX sch RC
Parts:
- removed Q?: IRLML6401, SOT:SOT23-3, symbol P_3PIN
- removed R?: 10k, Resistors:RES_0603, symbol R
- removed SW?: BUTTON, BtnsSwitches:BTN_4x4_SMD, symbol BUTTON
- added D1: L-C191LBCT, LEDs:LED_0603, symbol LED
- added D3: PMEG2020, Diodes:SOD323, symbol D_Shottky
- added J1, J2: Joystick, symbol Joystick
- added R1: 51R, Resistors:RES_0603, symbol R
- added R3, R5: 1k, Resistors:RES_0603, symbol R
- added R6, R7: 10k, Resistors:VAR_PTV09A-4, symbol RVar
- added SW1, SW4, SW5, SW6, SW7, SW8: IT-1187A, BtnsSwitches:BTN_4x4_SMD, symbol BUTTON
- added SW2: DIPx8, symbol DIPx8
- added U2: BT_HC05, Modules:BT_HC0x, symbol BT_HC05
- added XL1: PLS-8, symbol CONN_8
- gave numbers to parts that had none: 56
Connections:
- net labels added: BTN_A, BTN_B, BTN_C, BTN_D, BTN_J1, BTN_J2, BTN_L, BT_PIO11, BT_RESET, DIP1, DIP2, DIP3, DIP4, DIP5, DIP6, DIP7, DIP8, LCD_BCKLT, LCD_CE, LCD_CLK, LCD_DC, LCD_DIN, LCD_RST, MCURX_BTTX, MCUTX_BTRX
- wire segments 184 -> 284
- no-connect marks 11 -> 20
Other:
- note added: "Bluetooth"
- note added: "Buttons"
- note added: "DIP Switch"
- note added: "Joysticks"
- note added: "LCD"
- note added: "Potentiometers"
- note added: "USB detect"

Commit message: TX layout started
Parts:
- added HOLE5, HOLE6, HOLE7, HOLE8: HOLE_METALLED, PCB:Hole3_5_out6mm, symbol HOLE_METALLED
- added Logo2: Logo, Pictures:Livetronic27x9, symbol Logo
- J1, J2: footprint (none) -> BtnsSwitches:Joystick
- SW2: footprint (none) -> BtnsSwitches:DIP_SMD_X8
- XL1: footprint (none) -> Connectors:PLS-8
Connections:
- no-connect marks 20 -> 24

Commit message: + Layout + antenna
Parts:
- removed ANT1: ANT_PCB_MONO, Radio:ANT_868_SEIDHE, symbol ANT_PCB_MONO
- added ANT1: ANT_PCB_MONO_2PIN, Radio:ANT_868_IFA_SIMPLEJOY, symbol ANT_PCB_MONO_2PIN
- added D4: L-C191KGCT, LEDs:LED_0603, symbol LED
- added D5: L-C191LBCT, LEDs:LED_0603, symbol LED
- added Logo3: Logo, Pictures:Livetronic27x9, symbol Logo
- added R12, R13: 1k, Resistors:RES_0603, symbol R
- SW3: footprint BtnsSwitches:SW_SS-1P2T -> BtnsSwitches:SW_SS-12F23
Connections:
- net labels removed: PwrMCU
- wire segments 284 -> 306
- no-connect marks 24 -> 18
Other:
- note added: "Link"

Commit message: + SimpleJoy TX * Leg 63 bug fixed
Parts:
- added RP1, RP2, RP3, RP4: REFPOINT, PCB:REF_POINT_1MM, symbol REFPOINT
Changed lines of the file:
@@
 Wire Wire Line
 	15200 1800 15200 2450
+$Comp
+L REFPOINT RP1
+U 1 1 59DE1E3F
+P 13650 8350
+F 0 "RP1" H 13778 8403 60  0000 L CNN
+F 1 "REFPOINT" H 13778 8297 60  0000 L CNN
+F 2 "PCB:REF_POINT_1MM" H 13650 8350 60  0001 C CNN
+F 3 "" H 13650 8350 60  0000 C CNN
+	1    13650 8350
+	1    0    0    -1
+$EndComp
+$Comp
+L REFPOINT RP2
+U 1 1 59DE2203
+P 13650 8600
+F 0 "RP2" H 13778 8653 60  0000 L CNN
+F 1 "REFPOINT" H 13778 8547 60  0000 L CNN
+F 2 "PCB:REF_POINT_1MM" H 13650 8600 60  0001 C CNN
+F 3 "" H 13650 8600 60  0000 C CNN
+	1    13650 8600
+	1    0    0    -1
+$EndComp
+$Comp
+L REFPOINT RP3
+U 1 1 59DE2349
+P 13650 8850
+F 0 "RP3" H 13778 8903 60  0000 L CNN
+F 1 "REFPOINT" H 13778 8797 60  0000 L CNN
+F 2 "PCB:REF_POINT_1MM" H 13650 8850 60  0001 C CNN
+F 3 "" H 13650 8850 60  0000 C CNN
+	1    13650 8850
+	1    0    0    -1
+$EndComp
+$Comp
+L REFPOINT RP4
+U 1 1 59DE234F
+P 13650 9100
+F 0 "RP4" H 13778 9153 60  0000 L CNN
+F 1 "REFPOINT" H 13778 9047 60  0000 L CNN
+F 2 "PCB:REF_POINT_1MM" H 13650 9100 60  0001 C CNN
+F 3 "" H 13650 9100 60  0000 C CNN
+	1    13650 9100
+	1    0    0    -1
+$EndComp
 $EndSCHEMATC

Commit message: + Antennas matched
Parts:
- C20: value * -> 2pF
- C23: value * -> DoNotMount
- L4: value * -> 1.2nH
Changed lines of the file:
@@
 P 14450 1700
 F 0 "L4" V 14350 1560 40  0000 C CNN
-F 1 "*" V 14350 1700 40  0000 C CNN
+F 1 "1.2nH" V 14350 1700 40  0000 C CNN
 F 2 "Inductors:IND_0402" V 14510 1710 40  0001 C CNN
 F 3 "" V 14350 1560 60  0001 C CNN
@@
 P 14100 2200
 F 0 "C20" H 14000 2100 50  0000 L CNN
-F 1 "*" H 14000 2300 50  0000 L CNN
+F 1 "2pF" H 14000 2300 50  0000 L CNN
 F 2 "Capacitors:CAP_0402" V 14200 2050 28  0001 C BNN
 F 3 "" H 14000 2100 60  0001 C CNN
@@
 P 14800 2200
 F 0 "C23" H 14700 2100 50  0000 L CNN
-F 1 "*" H 14700 2300 50  0000 L CNN
+F 1 "DoNotMount" H 14600 2300 50  0000 L CNN
 F 2 "Capacitors:CAP_0402" V 14900 2050 28  0001 C BNN
 F 3 "" H 14700 2100 60  0001 C CNN

Commit message: + RX v2
Parts:
- ANT1, Logo1, Logo2, Logo3, RP1, RP2, RP3, RP4, XL4: Price (none) -> 0; SolderPoints (none) -> 0
- B1: Price (none) -> 30; SolderPoints (none) -> 2; URL (none) -> http://www.quartz1.com/price/model.php?akt=5470.11
- BLN1: Price (none) -> 45
- C1, C17, R10, R11, R4, R8: Price (none) -> 0.5; SolderPoints (none) -> 2
- D2, D3: Price (none) -> 5; SolderPoints (none) -> 2
- L3: value BLM15AG102SN1 -> BLM15AG102; PN (none) -> BLM15AG102SN1; Price (none) -> 1; SolderPoints (none) -> 2
- Q1: Price (none) -> 1.6
- SW2: PN (none) -> 1-1825058-9; Price (none) -> 35; SolderPoints (none) -> 16; URL (none) -> https://www.terraelectronica.ru/catalog_info.php?CODE=854801
- U1: SolderPoints (none) -> 6
- XL1: value PLS-8 -> PBS-8; Price (none) -> 24; SolderPoints (none) -> 8; URL (none) -> http://www.quartz1.com/price/model.php?group=1136&ext=1932
- XL2: Price (none) -> 2; SolderPoints (none) -> 6; SolderPointsDIP 6 -> (none)
- XL3: PN (none) -> 47491-0001; Price (none) -> 46; SolderPoints (none) -> 9
Changed lines of the file:
@@
 F 2 "Resistors:RES_0603" H 5950 4750 60  0001 C CNN
 F 3 "" H 5950 4750 60  0001 C CNN
+F 4 "2" V 5950 4750 60  0001 C CNN "SolderPoints"
+F 5 "0.5" V 5950 4750 60  0001 C CNN "Price"
 	1    5950 4750
 	1    0    0    -1
@@
 F 2 "Capacitors:CAP_0603" V 1650 7350 28  0001 C BNN
 F 3 "" H 1700 7500 60  0000 C CNN
+F 4 "2" H 1700 7500 60  0001 C CNN "SolderPoints"
+F 5 "0.5" H 1700 7500 60  0001 C CNN "Price"
 	1    1700 7500
 	1    0    0    -1
@@
 F 2 "Connectors:USBmicro_MOLEX_WM17142" H 1350 8000 60  0001 C CNN
 F 3 "" H 1350 8000 60  0000 C CNN
+F 4 "47491-0001" H 1350 8000 60  0001 C CNN "PN"
+F 5 "9" H 1350 8000 60  0001 C CNN "SolderPoints"
+F 6 "46" H 1350 8000 60  0001 C CNN "Price"
 	1    1350 8000
 	1    0    0    -1
@@
 F 2 "Connectors:PLS-6" H 1250 6000 60  0001 C CNN
 F 3 "" H 1250 6000 60  0000 C CNN
-F 4 "6" V 1250 6000 60  0001 C CNN "SolderPointsDIP"
+F 4 "6" V 1250 6000 60  0001 C CNN "SolderPoints"
+F 5 "2" V 1250 6000 60  0001 C CNN "Price"
 	1    1250 6000
 	-1   0    0    -1
@@
 F 5 "http://onelec.ru/products/0896bm15a0001e-52ab3408-7c12-4b8c-99ab-cc294cdc1e18" H 13000 2350 60  0001 C CNN "URL"
 F 6 "6" H 13100 2450 60  0001 C CNN "SolderPoints"
+F 7 "45" H 13150 1800 60  0001 C CNN "Price"
 	1    13150 1800
 	1    0    0    -1
@@
 	15150 4500 15150 4600
 $Comp
-L L L3
-U 1 1 59D40A02
-P 13050 4000
-F 0 "L3" V 12900 3850 40  0000 C CNN
-F 1 "BLM15AG102SN1" V 12950 4000 40  0000 C CNN
-F 2 "Inductors:IND_0402" V 13110 4010 40  0001 C CNN
-F 3 "" H 13050 4000 60  0000 C CNN
-	1    13050 4000
-	0    1    1    0
-$EndComp
-$Comp
 L GND #PWR067
 U 1 1 59D40A09
@@
 	1    0    0    -1
 $EndComp
-$Comp
-L C C17
-U 1 1 59D40A0F
-P 13350 4300
-F 0 "C17" H 13250 4400 50  0000 L CNN
-F 1 "1u" H 13250 4200 50  0000 L CNN
-F 2 "Capacitors:CAP_0603" H 13350 4300 60  0001 C CNN
-F 3 "" H 13350 4300 60  0001 C CNN
-	1    13350 4300
-	1    0    0    -1
-$EndComp
 Wire Wire Line
 	13350 4500 13350 4600
@@
 F 5 "9" H 1450 10150 60  0001 C CNN "Price"
 F 6 "https://www.terraelectronica.ru/catalog_info.php?CODE=244787" H 1550 10250 60  0001 C CNN "URL"
+F 7 "6" H 1600 9650 60  0001 C CNN "SolderPoints"
 	1    1600 9650
 	1    0    0    -1
@@
 $EndComp
 $Comp
-L C C10
-U 1 1 59D48A1B
-P 4000 4750
-F 0 "C10" H 3900 4650 50  0000 L CNN
-F 1 "10n" H 3900 4850 50  0000 L CNN
-F 2 "Capacitors:CAP_0603" V 4100 4600 28  0001 C BNN
-F 3 "" H 3900 4650 60  0001 C CNN
-F 4 "0.5" H 4000 4750 60  0001 C CNN "Price"
-F 5 "2" H 4100 4850 60  0001 C CNN "SolderPoints"
-	1    4000 4750
-	1    0    0    -1
-$EndComp
-$Comp
 L C C11
 U 1 1 59D48AE3
@@
 F 2 "Installation:BATTERY_AAA_X3" H 4150 10550 60  0001 C CNN
 F 3 "" H 4150 10550 60  0000 C CNN
+F 4 "2" H 4150 10550 60  0001 C CNN "SolderPoints"
+F 5 "http://www.quartz1.com/price/model.php?akt=5470.11" H 4150 10550 60  0001 C CNN "URL"
+F 6 "30" H 4150 10550 60  0001 C CNN "Price"
 	1    4150 10550
 	1    0    0    -1
@@
 $EndComp
 $Comp
-L R R10
-U 1 1 59D4DCFB
-P 9750 9000
-F 0 "R10" V 9830 9000 50  0000 C CNN
-F 1 "100k" V 9750 9000 50  0000 C CNN
-F 2 "Resistors:RES_0603" H 9750 9000 60  0001 C CNN
-F 3 "" H 9750 9000 60  0001 C CNN
-	1    9750 9000
-	1    0    0    -1
-$EndComp
-$Comp
-L R R11
-U 1 1 59D4DD02
-P 9750 9650
-F 0 "R11" V 9830 9650 50  0000 C CNN
-F 1 "100k" V 9750 9650 50  0000 C CNN
-F 2 "Resistors:RES_0603" H 9750 9650 60  0001 C CNN
-F 3 "" H 9750 9650 60  0001 C CNN
-	1    9750 9650
-	1    0    0    -1
-$EndComp
-$Comp
 L D_Shottky D2
 U 1 1 59D4DD09
@@
 F 2 "Diodes:SOD323" H 4550 8900 60  0001 C CNN
 F 3 "" H 4550 8900 60  0000 C CNN
+F 4 "2" H 4550 8900 60  0001 C CNN "SolderPoints"
+F 5 "5" H 4550 8900 60  0001 C CNN "Price"
 	1    4550 8900
 	1    0    0    -1
@@
 F 2 "Resistors:RES_0603" H 9400 10550 60  0001 C CNN
 F 3 "" H 9400 10550 60  0001 C CNN
+F 4 "2" V 9400 10550 60  0001 C CNN "SolderPoints"
+F 5 "0.5" V 9400 10550 60  0001 C CNN "Price"
 	1    9400 10550
 	-1   0    0    1
@@
 F 3 "" H 2000 -4350 60  0001 C CNN
 F 4 "3" H 2100 -4250 60  0001 C CNN "SolderPoints"
+F 5 "1.6" H 9700 10150 60  0001 C CNN "Price"
 	1    9700 10150
 	1    0    0    1
@@
 F 2 "Connectors:PLS-1Rnd" H -3500 -4400 60  0001 C CNN
 F 3 "" H -3500 -4400 60  0000 C CNN
+F 4 "0" H 13800 9550 60  0001 C CNN "SolderPoints"
+F 5 "0" H 13800 9550 60  0001 C CNN "Price"
 	1    13800 9550
 	1    0    0    -1
@@
 F 2 "Pictures:Ostranna_12d7_10d1" H 11300 8800 60  0001 C CNN
 F 3 "" H 11300 8800 60  0000 C CNN
+F 4 "0" H 11300 8800 60  0001 C CNN "SolderPoints"
+F 5 "0" H 11300 8800 60  0001 C CNN "Price"
 	1    11300 8800
 	1    0    0    -1
@@
 F 2 "BtnsSwitches:DIP_SMD_X8" H 6950 6800 60  0001 C CNN
 F 3 "" H 6950 6800 60  0000 C CNN
+F 4 "1-1825058-9" H 6950 6800 60  0001 C CNN "PN"
+F 5 "16" H 6950 6800 60  0001 C CNN "SolderPoints"
+F 6 "35" H 6950 6800 60  0001 C CNN "Price"
+F 7 "https://www.terraelectronica.ru/catalog_info.php?CODE=854801" H 6950 6800 60  0001 C CNN "URL"
 	1    6950 6800
 	1    0    0    -1
@@
 	0    1    1    0
 $EndComp
-$Comp
-L D_Shottky D3
-U 1 1 59D96630
-P 4550 9350
-F 0 "D3" H 4550 9450 40  0000 C CNN
-F 1 "PMEG2020" H 4550 9250 40  0000 C CNN
-F 2 "Diodes:SOD323" H 4550 9350 60  0001 C CNN
-F 3 "" H 4550 9350 60  0000 C CNN
-	1    4550 9350
-	1    0    0    -1
-$EndComp
 Wire Wire Line
 	4350 8900 4000 8900
@@
 P 1100 1450
 F 0 "XL1" H 1150 2000 50  0000 L CNN
-F 1 "PLS-8" H 1050 1900 50  0000 L CNN
+F 1 "PBS-8" H 1050 1900 50  0000 L CNN
 F 2 "Connectors:PLS-8" H 1100 1450 60  0001 C CNN
 F 3 "" H 1100 1450 60  0000 C CNN
+F 4 "http://www.quartz1.com/price/model.php?group=1136&ext=1932" H 1100 1450 60  0001 C CNN "URL"
+F 5 "24" H 1100 1450 60  0001 C CNN "Price"
+F 6 "8" H 1100 1450 60  0001 C CNN "SolderPoints"
 	1    1100 1450
 	-1   0    0    -1
@@
 F 2 "Pictures:Livetronic27x9" H 11300 9800 60  0001 C CNN
 F 3 "" H 11300 9800 60  0000 C CNN
+F 4 "0" H 11300 9800 60  0001 C CNN "SolderPoints"
+F 5 "0" H 11300 9800 60  0001 C CNN "Price"
 	1    11300 9800
 	1    0    0    -1
@@
 F 2 "Pictures:Livetronic27x9" H 11300 10800 60  0001 C CNN
 F 3 "" H 11300 10800 60  0000 C CNN
+F 4 "0" H 11300 10800 60  0001 C CNN "SolderPoints"
+F 5 "0" H 11300 10800 60  0001 C CNN "Price"
 	1    11300 10800
 	1    0    0    -1
@@
 F 2 "Radio:ANT_868_IFA_SIMPLEJOY" H 15400 1750 60  0001 C CNN
 F 3 "" H 15400 1750 60  0000 C CNN
+F 4 "0" H 15400 1750 60  0001 C CNN "SolderPoints"
+F 5 "0" H 15400 1750 60  0001 C CNN "Price"
 	1    15400 1750
 	1    0    0    -1
@@
 F 2 "PCB:REF_POINT_1MM" H 13650 8350 60  0001 C CNN
 F 3 "" H 13650 8350 60  0000 C CNN
+F 4 "0" H 13650 8350 60  0001 C CNN "SolderPoints"
+F 5 "0" H 13650 8350 60  0001 C CNN "Price"
 	1    13650 8350
 	1    0    0    -1
@@
 F 2 "PCB:REF_POINT_1MM" H 13650 8600 60  0001 C CNN
 F 3 "" H 13650 8600 60  0000 C CNN
+F 4 "0" H 13650 8600 60  0001 C CNN "SolderPoints"
+F 5 "0" H 13650 8600 60  0001 C CNN "Price"
 	1    13650 8600
 	1    0    0    -1
 $EndComp
 $Comp
+L C C10
+U 1 1 5A01A809
+P 4000 4750
+F 0 "C10" H 3950 4650 50  0000 L CNN
+F 1 "10n" H 3950 4850 50  0000 L CNN
+F 2 "Capacitors:CAP_0603" V 3950 4600 28  0001 C BNN
+F 3 "" H 4000 4750 60  0000 C CNN
+F 4 "2" H 4000 4750 60  0001 C CNN "SolderPoints"
+F 5 "0.5" H 4000 4750 60  0001 C CNN "Price"
+	1    4000 4750
+	1    0    0    -1
+$EndComp
+$Comp
+L C C17
+U 1 1 5A01C079
+P 13350 4300
+F 0 "C17" H 13250 4200 50  0000 L CNN
+F 1 "1u" H 13250 4400 50  0000 L CNN
+F 2 "Capacitors:CAP_0603" V 13450 4150 28  0001 C BNN
+F 3 "" H 13250 4200 60  0001 C CNN
+F 4 "0.5" H 13350 4300 60  0001 C CNN "Price"
+F 5 "2" H 13450 4400 60  0001 C CNN "SolderPoints"
+	1    13350 4300
+	1    0    0    -1
+$EndComp
+$Comp
+L D_Shottky D3
+U 1 1 5A01CF81
+P 4550 9350
+F 0 "D3" H 4550 9450 40  0000 C CNN
+F 1 "PMEG2020" H 4550 9250 40  0000 C CNN
+F 2 "Diodes:SOD323" H 4550 9350 60  0001 C CNN
+F 3 "" H 4550 9350 60  0000 C CNN
+F 4 "2" H 4550 9350 60  0001 C CNN "SolderPoints"
+F 5 "5" H 4550 9350 60  0001 C CNN "Price"
+	1    4550 9350
+	1    0    0    -1
+$EndComp
+$Comp
+L L L3
+U 1 1 5A01E638
+P 13050 4000
+F 0 "L3" V 12850 3850 40  0000 C CNN
+F 1 "BLM15AG102" V 12950 4000 40  0000 C CNN
+F 2 "Inductors:IND_0402" V 13110 4010 40  0001 C CNN
+F 3 "" V 12950 3860 60  0001 C CNN
+F 4 "1" V 13050 3960 60  0001 C CNN "Price"
+F 5 "2" V 13150 4060 60  0001 C CNN "SolderPoints"
+F 6 "BLM15AG102SN1" V 13050 4000 60  0001 C CNN "PN"
+	1    13050 4000
+	0    1    1    0
+$EndComp
+$Comp
+L R R10
+U 1 1 5A01FFE2
+P 9750 9000
+F 0 "R10" V 9830 9000 50  0000 C CNN
+F 1 "100k" V 9750 9000 50  0000 C CNN
+F 2 "Resistors:RES_0603" H 9750 9000 60  0001 C CNN
+F 3 "" H 9750 9000 60  0001 C CNN
+F 4 "2" V 9750 9000 60  0001 C CNN "SolderPoints"
+F 5 "0.5" V 9750 9000 60  0001 C CNN "Price"
+	1    9750 9000
+	-1   0    0    1
+$EndComp
+$Comp
+L R R11
+U 1 1 5A020478
+P 9750 9650
+F 0 "R11" V 9830 9650 50  0000 C CNN
+F 1 "100k" V 9750 9650 50  0000 C CNN
+F 2 "Resistors:RES_0603" H 9750 9650 60  0001 C CNN
+F 3 "" H 9750 9650 60  0001 C CNN
+F 4 "2" V 9750 9650 60  0001 C CNN "SolderPoints"
+F 5 "0.5" V 9750 9650 60  0001 C CNN "Price"
+	1    9750 9650
+	-1   0    0    1
+$EndComp
+$Comp
 L REFPOINT RP3
-U 1 1 59DE2349
+U 1 1 5A021EC6
 P 13650 8850
 F 0 "RP3" H 13778 8903 60  0000 L CNN
@@
 F 2 "PCB:REF_POINT_1MM" H 13650 8850 60  0001 C CNN
 F 3 "" H 13650 8850 60  0000 C CNN
+F 4 "0" H 13650 8850 60  0001 C CNN "SolderPoints"
+F 5 "0" H 13650 8850 60  0001 C CNN "Price"
 	1    13650 8850
 	1    0    0    -1
@@
 $Comp
 L REFPOINT RP4
-U 1 1 59DE234F
+U 1 1 5A021ECE
 P 13650 9100
 F 0 "RP4" H 13778 9153 60  0000 L CNN
@@
 F 2 "PCB:REF_POINT_1MM" H 13650 9100 60  0001 C CNN
 F 3 "" H 13650 9100 60  0000 C CNN
+F 4 "0" H 13650 9100 60  0001 C CNN "SolderPoints"
+F 5 "0" H 13650 9100 60  0001 C CNN "Price"
 	1    13650 9100
 	1    0    0    -1

Commit message: Proceeding
Parts:
- added C26: 100pF, Capacitors:CAP_0402, symbol Tittar_kl:C
- added J3, J4: Joystick, BtnsSwitches:JoystickSmall, symbol Switches:Joystick
- ANT1: symbol ANT_PCB_MONO_2PIN -> Antennas_kl:ANT_PCB_MONO_2PIN
- B1: symbol BAT -> Power_kl:BAT
- BLN1: symbol BALUN868JOHANSON -> RFICs:BALUN868JOHANSON
- C1, C10, C11, C12, C13, C14, C15, C16, C17, C18, C19, C2, C20, C21, C22, C23, C24, C25, C3, C4, C5, C6, C7, C8, C9: symbol C -> Tittar_kl:C
- D1, D4, D5: symbol LED -> Tittar_kl:LED
- D2, D3: symbol D_Shottky -> Tittar_kl:D_Shottky
- DA1: footprint SOT:SOT23-3 -> SOT:SOT23-3A; symbol MCP1700 -> Power_kl:MCP1700
- DD1: symbol STM32F072RxTx -> st_kl:STM32F072RxTx
- DD2: symbol CC1101 -> RFICs:CC1101
- HOLE1, HOLE2, HOLE3, HOLE4, HOLE5, HOLE6, HOLE7, HOLE8: symbol HOLE_METALLED -> pcb_details:HOLE_METALLED
- J1, J2: symbol Joystick -> Switches:Joystick
- L1, L2, L3, L4: symbol L -> Tittar_kl:L
- Logo1, Logo2, Logo3: symbol Logo -> pcb_details:Logo
- Q1: symbol N_3PIN -> Transistors_kl:N_3PIN
- R1, R10, R11, R12, R13, R2, R3, R4, R5, R8, R9: symbol R -> Tittar_kl:R
- R6, R7: symbol RVar -> Tittar_kl:RVar
- RP1, RP2, RP3, RP4: symbol REFPOINT -> pcb_details:REFPOINT
- SW1, SW4, SW5, SW6, SW7, SW8: symbol BUTTON -> Switches:BUTTON
- SW2: symbol DIPx8 -> Switches:DIPx8
- SW3: symbol SWITCH -> Switches:SWITCH
- TP1: symbol TESTPOINT -> pcb_details:TESTPOINT
- U1: symbol USBLC6 -> ESDProtection:USBLC6
- U2: symbol BT_HC05 -> modules:BT_HC05
- XL1: symbol CONN_8 -> Connectors_kl:CONN_8
- XL2: symbol CONN_6 -> Connectors_kl:CONN_6
- XL3: symbol USB_MINI_B -> Connectors_kl:USB_MINI_B
- XL4: symbol CONN_1 -> Connectors_kl:CONN_1
- XTAL1, XTAL2: symbol CRYSTAL_H -> Tittar_kl:CRYSTAL_H
Connections:
- wire segments 306 -> 404
- no-connect marks 18 -> 26
Other:
- note added: "Other footprint"
